Commit message: Try to add gazebo support.

File: src/moving_car/urdf/moving_car.urdf (robot description, URDF)
Before this commit: robot mvcar, 2 links, 1 joints
Links:
- added link camera_link; collision box size=0.01 0.01 0.01; visual box size=0.01 0.01 0.01
- link body_link: mass None -> 1.0; geometry collision mesh filename=package://moving_car/meshes/body.stl scale=0.001 0.001 0.001; visual mesh filename=package://moving_car/meshes/body.stl scale=0.001 0.001 0.001
Joints:
- added joint camera_joint: type fixed, parent body_link, child camera_link, origin xyz=0.0 0.08 0.045 rpy=-0.7853981633974483 0.0 0.0

Commit message: Fix meshes file path issue.

File: src/moving_car/urdf/moving_car.urdf (robot description, URDF)
Before this commit: robot mvcar, 3 links, 2 joints
Links:
- removed link dummy_link
- link body_link: geometry collision mesh filename=$(find moving_car)/meshes/body.stl scale=0.001 0.001 0.001; visual mesh filename=$(find moving_car)/meshes/body.stl scale=0.001 0.001 0.001
Joints:
- removed joint dummy_joint

Commit message: Add lidar, camera and imu sensors.

File: src/moving_car/urdf/moving_car.urdf (robot description, URDF)
Before this commit: robot mvcar, 2 links, 1 joints
Links:
- added link imu_link; collision box size=0.01 0.01 0.002; visual box size=0.01 0.01 0.002
- added link lidar_link; collision cylinder length=0.06 radius=0.005; visual cylinder length=0.06 radius=0.005
Joints:
- added joint imu_joint: type fixed, parent body_link, child imu_link, origin xyz=0.0 0.0 0.008 rpy=0.0 0.0 0.0
- added joint lidar_joint: type fixed, parent body_link, child lidar_link, origin xyz=0.0 0.06 0.03 rpy=0.0 0.0 0.0

Commit message: Implements comunication between ros and gazebo.

File: src/moving_car/urdf/moving_car.urdf (robot description, URDF)
Before this commit: robot mvcar, 4 links, 3 joints
Joints:
- joint camera_joint: origin xyz=0.0 0.08 0.045 rpy=-0.7853981633974483 0.0 0.0 -> xyz=0.0 0.077 0.045 rpy=0 0.0 0.0

Commit message: Fix physics propeties of the links, add diff_drive support.

File: src/moving_car/urdf/moving_car.urdf (robot description, URDF)
Before this commit: robot mvcar, 4 links, 3 joints
Links:
- link body_link: mass 1.0 -> ${body_mass}

Commit message: Fix camera link orientation.

File: src/moving_car/urdf/moving_car.urdf (robot description, URDF)
Before this commit: robot mvcar, 4 links, 3 joints
Links:
- link camera_link: geometry collision box size=0.001 0.02 0.01; visual box size=0.001 0.02 0.01
Joints:
- joint camera_joint: origin xyz=0.0 0.077 0.045 rpy=0 0.0 0.0 -> xyz=0.0 0.08 0.08 rpy=0.0 0.7853981633974483 1.5707963267948966
